Commit message: trying to visualize odometry in rviz

File: wheebbot_description/urdf/gazebo_spec_tags.xacro (robot description, xacro)
@@ -1,7 +1,8 @@
 <?xml version="1.0"?>
 <robot xmlns:xacro="http://www.ros.org/wiki/xacro">
-  <!-- ########### MODEL PLUGINS ############ -->
-  <!-- Model control plugin/s -->
-  <!-- <plugin name="libcontrol_plugin" filename="package://wheebbot/plugins/gazebo_classic/wheebbot_test/libcontrol_plugin.so"/> -->
+  <xacro:property name="yaml_file" value="$(find wheebbot_description)/config/urdf_params.yaml" />
+  <xacro:property name="props" value="${load_yaml(yaml_file)}"/>
+  <xacro:property name="wheels_interax" value="${props['wheebbot']['wheels_interax']}" />
+  <xacro:property name="wheels_diameter" value="${2* props['wheebbot']['wheel_radius']}" />
   <!-- joint state publisher (this way gazebo publishes joint states to RViz) -->
   <gazebo>
@@ -19,4 +20,71 @@
     <kp value="${body_kp_gazebo}" />
     <kd value="${body_kd_gazebo}" />
+    <!-- <sensor name="imu_sensor" type="imu">
+      <plugin filename="libgazebo_ros_imu_sensor.so" name="imu_plugin">
+         <ros>
+           <namespace></namespace>
+           <remapping>~/out:=imu</remapping>
+         </ros>
+         <initial_orientation_as_reference>false</initial_orientation_as_reference>
+       </plugin>
+       <always_on>true</always_on>
+       <update_rate>100</update_rate>
+       <visualize>true</visualize>
+       <imu>
+         <angular_velocity>
+           <x>
+             <noise type="gaussian">
+               <mean>0.0</mean>
+               <stddev>0.0</stddev>
+               <bias_mean>0.0</bias_mean>
+               <bias_stddev>0.0</bias_stddev>
+             </noise>
+           </x>
+           <y>
+             <noise type="gaussian">
+               <mean>0.0</mean>
+               <stddev>0.0</stddev>
+               <bias_mean>0.0</bias_mean>
+               <bias_stddev>0.0</bias_stddev>
+             </noise>
+           </y>
+           <z>
+             <noise type="gaussian">
+               <mean>0.0</mean>
+               <stddev>0.0</stddev>
+               <bias_mean>0.0</bias_mean>
+               <bias_stddev>0.0</bias_stddev>
+             </noise>
+           </z>
+         </angular_velocity>
+         <linear_acceleration>
+           <x>
+             <noise type="gaussian">
+               <mean>0.0</mean>
+               <stddev>0.0</stddev>
+               <bias_mean>0.0</bias_mean>
+               <bias_stddev>0.0</bias_stddev>
+             </noise>
+           </x>
+           <y>
+             <noise type="gaussian">
+               <mean>0.0</mean>
+               <stddev>0.0</stddev>
+               <bias_mean>0.0</bias_mean>
+               <bias_stddev>0.0</bias_stddev>
+             </noise>
+           </y>
+           <z>
+             <noise type="gaussian">
+               <mean>0.0</mean>
+               <stddev>0.0</stddev>
+               <bias_mean>0.0</bias_mean>
+               <bias_stddev>0.0</bias_stddev>
+             </noise>
+           </z>
+         </linear_acceleration>
+       </imu>
+     </sensor>
+      -->
   </gazebo>
   <!-- right wheel -->
@@ -36,3 +104,26 @@
     <maxContacts value="${wheel_max_contacts_gazebo}" />
   </gazebo>
+  <!-- diff drive plugin -->
+  <!-- <gazebo>
+    <plugin name='diff_drive' filename='libgazebo_ros_diff_drive.so'>
+      <ros>
+        <namespace>/base_state</namespace>
+      </ros>
+      <!-- wheels -->
+      <left_joint>left_wheel_joint</left_joint>
+      <right_joint>right_wheel_joint</right_joint>
+      <!-- kinematics -->
+      <wheel_separation> 0.028</wheel_separation>
+      <wheel_diameter> 0.12 </wheel_diameter>
+      <!-- limits -->
+      <max_wheel_torque>2</max_wheel_torque>
+      <max_wheel_acceleration>1.0</max_wheel_acceleration>
+      <!-- output -->
+      <publish_odom>true</publish_odom>
+      <publish_odom_tf>false</publish_odom_tf>
+      <publish_wheel_tf>true</publish_wheel_tf>
+      <odometry_frame>world</odometry_frame>
+      <robot_base_frame>aux_link</robot_base_frame>
+    </plugin>
+  </gazebo> -->
 </robot>

File: wheebbot_description/urdf/wheebbot.urdf.xacro (robot description, xacro)
@@ -1,166 +1,167 @@
 <?xml version="1.0"?>
 <robot name="wheebbot" xmlns:xacro="http://www.ros.org/wiki/xacro">
-  <xacro:arg name="is_gazebo_classic" default="true" />
-  <xacro:property name="wheebbot_description_path" value="$(find wheebbot_description)"/>
-  <!-- Including the parameters file -->
-  <xacro:include filename="${wheebbot_description_path}/urdf/parameters.urdf.xacro" />
-  <!-- Including the macros file -->
-  <xacro:include filename="${wheebbot_description_path}/urdf/macros.urdf.xacro" />
-  <!-- Including the materials file -->
-  <!-- <xacro:include filename="${wheebbot_description_path}/urdf/materials.urdf.xacro" /> -->
-  <xacro:if value="$(arg is_gazebo_classic)">
-    <!-- Including the gazebo related stuff -->
-    <xacro:include filename="${wheebbot_description_path}/urdf/gazebo_spec_tags.xacro" />
-  </xacro:if>
-  <xacro:unless value="$(arg is_gazebo_classic)">
-    <!-- Including the gazebo related stuff -->
-    <xacro:include filename="${wheebbot_description_path}/urdf/ign_spec_tags.xacro" />
-  </xacro:unless>
-  <link name="aux_link">
-  </link>
-  <link name="body">
-    <!-- body visual -->
-    <visual>
-      <origin xyz="0 ${box_ly/2-leg_extrusion_l_edge/2} ${-(box_lz/2-leg_extrusion_l_edge/2)}" rpy="0 0 ${-pi/2}" />
-      <geometry>
-        <mesh filename="package://wheebbot_description/meshes/full_no_knee_no_wheels.dae" scale="1.0 1.0 1.0" />
-      </geometry>
-    </visual>
-    <!-- box -->
-    <collision>
-      <origin xyz="0 0 0" rpy="0 0 0"/>
+  <xacro:macro name="ign_or_gazebo" params="is_gazebo_classic" >
+    <!-- Including the parameters file -->
+    <xacro:include filename="$(find wheebbot_description)/urdf/parameters.urdf.xacro" />
+    <!-- Including the macros file -->
+    <xacro:include filename="$(find wheebbot_description)/urdf/macros.urdf.xacro" />
+    <!-- Including the materials file -->
+    <!-- <xacro:include filename="$(find wheebbot_description)/urdf/materials.urdf.xacro" /> -->
+    <xacro:if value="${is_gazebo_classic}">
+      <!-- Including the gazebo related stuff -->
+      <xacro:include filename="$(find wheebbot_description)/urdf/gazebo_spec_tags.xacro" />
+    </xacro:if>
+    <xacro:unless value="${is_gazebo_classic}">
+      <!-- Including the gazebo related stuff -->
+      <xacro:include filename="$(find wheebbot_description)/urdf/ign_spec_tags.xacro" />
+    </xacro:unless>
+    <!-- auxiliary link on the ground (fixed wrt the robot) -->
+    <link name="aux_link">
+    </link>
+    <joint name="aux_joint" type="fixed">
+      <origin xyz="0 0 ${(box_lz/2+leg_length+motor_case_l_edge/2+wheel_radius)}" rpy="0 0 0"/>
+      <parent link="aux_link"/>
+      <child link="body"/>
+    </joint>
+    <link name="body">
+      <!-- body visual -->
+      <visual>
+        <origin xyz="0 ${box_ly/2-leg_extrusion_l_edge/2} ${-(box_lz/2-leg_extrusion_l_edge/2)}" rpy="0 0 ${-pi/2}" />
         <geometry>
-          <box size="${box_lx} ${box_ly} ${box_lz}" />
+          <mesh filename="package://wheebbot_description/meshes/full_no_knee_no_wheels.dae" scale="1.0 1.0 1.0" />
         </geometry>
-    </collision>
-   <!-- top fan collision group-->
-   <!-- fan-->
-    <collision>
-      <origin xyz="0 0 ${(box_lz/2+fan_vert_footprint/2)}" rpy="0 0 0"/>
+      </visual>
+      <!-- box -->
+      <collision>
+        <origin xyz="0 0 0" rpy="0 0 0"/>
+          <geometry>
+            <box size="${box_lx} ${box_ly} ${box_lz}" />
+          </geometry>
+      </collision>
+    <!-- top fan collision group-->
+    <!-- fan-->
+      <collision>
+        <origin xyz="0 0 ${(box_lz/2+fan_vert_footprint/2)}" rpy="0 0 0"/>
+          <geometry>
+            <box size="${fan_edge_length} ${fan_edge_length} ${fan_vert_footprint}" />
+          </geometry>
+      </collision>
+      <!-- left door handle-->
+      <collision>
+        <origin xyz="0 ${box_ly/2-door_handle_width/2} ${(box_lz/2+door_handle_height2/2)}" rpy="0 0 0"/>
+          <geometry>
+            <box size="${door_handle_tot_lenght} ${door_handle_width} ${door_handle_height2}" />
+          </geometry>
+      </collision>
+      <collision>
+        <origin xyz="0 ${box_ly/2-door_handle_width/2} ${(box_lz/2+door_handle_height2+(door_handle_tot_height-door_handle_height2)/2)}" rpy="0 0 0"/>
+          <geometry>
+            <box size="${door_handle_lenght2} ${door_handle_width} ${door_handle_tot_height-door_handle_height2}" />
+          </geometry>
+      </collision>
+      <!-- right door handle-->
+      <collision>
+        <origin xyz="0 ${-(box_ly/2-door_handle_width/2)} ${(box_lz/2+door_handle_height2/2)}" rpy="0 0 0"/>
+          <geometry>
+            <box size="${door_handle_tot_lenght} ${door_handle_width} ${door_handle_height2}" />
+          </geometry>
+      </collision>
+      <collision>
+        <origin xyz="0 ${-(box_ly/2-door_handle_width/2)} ${(box_lz/2+door_handle_height2+(door_handle_tot_height-door_handle_height2)/2)}" rpy="0 0 0"/>
+          <geometry>
+            <box size="${door_handle_lenght2} ${door_handle_width} ${door_handle_tot_height-door_handle_height2}" />
+          </geometry>
+      </collision>
+      <!-- back fan collision -->
+      <collision>
+        <origin xyz="${-(box_lx/2+fan_vert_footprint/2)} 0 0" rpy="0 ${-pi/2} 0"/>
+          <geometry>
+            <box size="${fan_edge_length} ${fan_edge_length} ${fan_vert_footprint}" />
+          </geometry>
+      </collision>
+      <!-- left leg -->
+      <collision>
+        <origin xyz="${(leg_pos_wrt_box_back-box_lx/2)} ${box_ly/2-leg_extrusion_l_edge/2} ${-(box_lz/2+leg_length/2)}" rpy="0 0 0"/>
+          <geometry>
+            <box size="${leg_extrusion_l_edge} ${leg_extrusion_l_edge} ${leg_length}" />
+          </geometry>
+      </collision>
+      <!-- left motor case -->
+      <collision>
+        <origin xyz="${(leg_pos_wrt_box_back-box_lx/2)} ${box_ly/2-motor_case_extension/2} ${-(box_lz/2+leg_length+motor_case_l_edge/2)}" rpy="0 0 0"/>
+          <geometry>
+            <box size="${motor_case_l_edge} ${motor_case_extension} ${motor_case_l_edge}" />
+          </geometry>
+      </collision>
+      <!-- right leg -->
+      <collision>
+        <origin xyz="${(leg_pos_wrt_box_back-box_lx/2)} ${-(box_ly/2-leg_extrusion_l_edge/2)} ${-(box_lz/2+leg_length/2)}" rpy="0 0 0"/>
+          <geometry>
+            <box size="${leg_extrusion_l_edge} ${leg_extrusion_l_edge} ${leg_length}" />
+          </geometry>
+      </collision>
+      <!-- right motor case -->
+      <collision>
+        <origin xyz="${(leg_pos_wrt_box_back-box_lx/2)} ${-(box_ly/2-motor_case_extension/2)} ${-(box_lz/2+leg_length+motor_case_l_edge/2)}" rpy="0 0 0"/>
+          <geometry>
+            <box size="${motor_case_l_edge} ${motor_case_extension} ${motor_case_l_edge}" />
+          </geometry>
+      </collision>
+      <xacro:box_inertia mass="${pendulum_mass}" l_x="${pendulum_depth}" l_y="${pendulum_width}" l_z="${pendulum_length}">
+        <origin xyz="${pendulum_length*sin(pendulum_CoM_pitch_offset)} 0 ${-(box_lz/2+leg_length+motor_case_l_edge/2)+pendulum_length*cos(pendulum_CoM_pitch_offset)}" rpy="0 ${pendulum_CoM_pitch_offset} 0"/>
+      </xacro:box_inertia>
+    </link>
+    <joint name="left_wheel_joint" type="continuous">
+      <origin xyz="0 ${(wheels_interax/2)} ${-(box_lz/2+leg_length+motor_case_l_edge/2)}" rpy="0 0 0"/>
+      <parent link="body"/>
+      <child link="left_wheel"/>
+      <axis xyz="0 1 0" />
+      <dynamics damping="${wheel_joint_damping}" friction="${wheel_joint_static_friction}"/>
+      <limit effort="${wheel_joint_effort_lim}" velocity="${wheel_joint_velocity_lim}" />
+    </joint>
+    <link name="left_wheel">
+      <!-- wheel visual -->
+      <visual>
+        <origin xyz="0 0 0" rpy="0 0 ${pi/2}" />
         <geometry>
-          <box size="${fan_edge_length} ${fan_edge_length} ${fan_vert_footprint}" />
+          <mesh filename="package://wheebbot_description/meshes/wheel_black.dae" scale="1.0 1.0 1.0" />
         </geometry>
-    </collision>
-    <!-- left door handle-->
-    <collision>
-      <origin xyz="0 ${box_ly/2-door_handle_width/2} ${(box_lz/2+door_handle_height2/2)}" rpy="0 0 0"/>
+      </visual>
+      <collision>
+        <origin xyz="0 0 0" rpy="${pi/2} 0 0"/>
+          <geometry>
+            <cylinder radius="${wheel_radius}" length="${wheel_thickness}"/>
+          </geometry>
+      </collision>
+      <xacro:disk_inertia mass="${wheel_mass}" radius="${wheel_radius}" height="${wheel_thickness}">
+        <origin xyz="0 0 0" rpy="${-pi/2} 0 0" />
+      </xacro:disk_inertia>
+    </link>
+    <joint name="right_wheel_joint" type="continuous">
+      <origin xyz="0 ${-(wheels_interax/2)} ${-(box_lz/2+leg_length+motor_case_l_edge/2)}" rpy="0 0 0"/>
+      <parent link="body"/>
+      <child link="right_wheel"/>
+      <axis xyz="0 1 0" />
+      <dynamics damping="${wheel_joint_damping}" friction="${wheel_joint_static_friction}"/>
+      <limit effort="${wheel_joint_effort_lim}" velocity="${wheel_joint_velocity_lim}" />
+    </joint>
+    <link name="right_wheel">
+      <!-- wheel visual -->
+      <visual>
+        <origin xyz="0 0 0" rpy="0 0 ${-pi/2}" />
         <geometry>
-          <box size="${door_handle_tot_lenght} ${door_handle_width} ${door_handle_height2}" />
+          <mesh filename="package://wheebbot_description/meshes/wheel_black.dae" scale="1.0 1.0 1.0" />
         </geometry>
-    </collision>
-    <collision>
-      <origin xyz="0 ${box_ly/2-door_handle_width/2} ${(box_lz/2+door_handle_height2+(door_handle_tot_height-door_handle_height2)/2)}" rpy="0 0 0"/>
-        <geometry>
-          <box size="${door_handle_lenght2} ${door_handle_width} ${door_handle_tot_height-door_handle_height2}" />
-        </geometry>
-    </collision>
-    <!-- right door handle-->
-    <collision>
-       <origin xyz="0 ${-(box_ly/2-door_handle_width/2)} ${(box_lz/2+door_handle_height2/2)}" rpy="0 0 0"/>
-         <geometry>
-           <box size="${door_handle_tot_lenght} ${door_handle_width} ${door_handle_height2}" />
-         </geometry>
-     </collision>
-     <collision>
-       <origin xyz="0 ${-(box_ly/2-door_handle_width/2)} ${(box_lz/2+door_handle_height2+(door_handle_tot_height-door_handle_height2)/2)}" rpy="0 0 0"/>
-         <geometry>
-           <box size="${door_handle_lenght2} ${door_handle_width} ${door_handle_tot_height-door_handle_height2}" />
-         </geometry>
-     </collision>
-    <!-- back fan collision -->
-    <collision>
-      <origin xyz="${-(box_lx/2+fan_vert_footprint/2)} 0 0" rpy="0 ${-pi/2} 0"/>
-        <geometry>
-          <box size="${fan_edge_length} ${fan_edge_length} ${fan_vert_footprint}" />
-        </geometry>
-    </collision>
-    <!-- left leg -->
-    <collision>
-      <origin xyz="${(leg_pos_wrt_box_back-box_lx/2)} ${box_ly/2-leg_extrusion_l_edge/2} ${-(box_lz/2+leg_length/2)}" rpy="0 0 0"/>
-        <geometry>
-          <box size="${leg_extrusion_l_edge} ${leg_extrusion_l_edge} ${leg_length}" />
-        </geometry>
-    </collision>
-    <!-- left motor case -->
-    <collision>
-      <origin xyz="${(leg_pos_wrt_box_back-box_lx/2)} ${box_ly/2-motor_case_extension/2} ${-(box_lz/2+leg_length+motor_case_l_edge/2)}" rpy="0 0 0"/>
-        <geometry>
-          <box size="${motor_case_l_edge} ${motor_case_extension} ${motor_case_l_edge}" />
-        </geometry>
-    </collision>
-    <!-- right leg -->
-    <collision>
-      <origin xyz="${(leg_pos_wrt_box_back-box_lx/2)} ${-(box_ly/2-leg_extrusion_l_edge/2)} ${-(box_lz/2+leg_length/2)}" rpy="0 0 0"/>
-        <geometry>
-          <box size="${leg_extrusion_l_edge} ${leg_extrusion_l_edge} ${leg_length}" />
-        </geometry>
-    </collision>
-    <!-- right motor case -->
-    <collision>
-      <origin xyz="${(leg_pos_wrt_box_back-box_lx/2)} ${-(box_ly/2-motor_case_extension/2)} ${-(box_lz/2+leg_length+motor_case_l_edge/2)}" rpy="0 0 0"/>
-        <geometry>
-          <box size="${motor_case_l_edge} ${motor_case_extension} ${motor_case_l_edge}" />
-        </geometry>
-    </collision>
-    <xacro:box_inertia mass="${pendulum_mass}" l_x="${pendulum_depth}" l_y="${pendulum_width}" l_z="${pendulum_length}">
-      <origin xyz="${pendulum_length*sin(pendulum_CoM_pitch_offset)} 0 ${-(box_lz/2+leg_length+motor_case_l_edge/2)+pendulum_length*cos(pendulum_CoM_pitch_offset)}" rpy="0 ${pendulum_CoM_pitch_offset} 0"/>
-    </xacro:box_inertia>
-  </link>
-  <link name="left_wheel">
-    <!-- wheel visual -->
-    <visual>
-      <origin xyz="0 0 0" rpy="0 0 ${pi/2}" />
-      <geometry>
-        <mesh filename="package://wheebbot_description/meshes/wheel_black.dae" scale="1.0 1.0 1.0" />
-      </geometry>
-    </visual>
-    <collision>
-      <origin xyz="0 0 0" rpy="${pi/2} 0 0"/>
-        <geometry>
-          <cylinder radius="${wheel_radius}" length="${wheel_thickness}"/>
-        </geometry>
-    </collision>
-    <xacro:disk_inertia mass="${wheel_mass}" radius="${wheel_radius}" height="${wheel_thickness}">
-      <origin xyz="0 0 0" rpy="${-pi/2} 0 0" />
-    </xacro:disk_inertia>
-  </link>
-  <link name="right_wheel">
-    <!-- wheel visual -->
-    <visual>
-      <origin xyz="0 0 0" rpy="0 0 ${-pi/2}" />
-      <geometry>
-        <mesh filename="package://wheebbot_description/meshes/wheel_black.dae" scale="1.0 1.0 1.0" />
-      </geometry>
-    </visual>
-    <collision>
-      <origin xyz="0 0 0" rpy="${pi/2} 0 0"/>
-        <geometry>
-          <cylinder radius="${wheel_radius}" length="${wheel_thickness}"/>
-        </geometry>
-    </collision>
-    <xacro:disk_inertia mass="${wheel_mass}" radius="${wheel_radius}" height="${wheel_thickness}">
-      <origin xyz="0 0 0" rpy="${-pi/2} 0 0" />
-    </xacro:disk_inertia >
-  </link>
-  <joint name="aux_joint" type="fixed">
-    <origin xyz="0 0 ${(box_lz/2+leg_length+motor_case_l_edge/2+wheel_radius)}" rpy="0 0 0"/>
-    <parent link="aux_link"/>
-    <child link="body"/>
-  </joint>
-  <joint name="left_wheel_joint" type="continuous">
-    <origin xyz="0 ${(wheels_interax/2)} ${-(box_lz/2+leg_length+motor_case_l_edge/2)}" rpy="0 0 0"/>
-    <parent link="body"/>
-    <child link="left_wheel"/>
-    <axis xyz="0 1 0" />
-    <dynamics damping="${wheel_joint_damping}" friction="${wheel_joint_static_friction}"/>
-    <limit effort="${wheel_joint_effort_lim}" velocity="${wheel_joint_velocity_lim}" />
-  </joint>
-  <joint name="right_wheel_joint" type="continuous">
-    <origin xyz="0 ${-(wheels_interax/2)} ${-(box_lz/2+leg_length+motor_case_l_edge/2)}" rpy="0 0 0"/>
-    <parent link="body"/>
-    <child link="right_wheel"/>
-    <axis xyz="0 1 0" />
-    <dynamics damping="${wheel_joint_damping}" friction="${wheel_joint_static_friction}"/>
-    <limit effort="${wheel_joint_effort_lim}" velocity="${wheel_joint_velocity_lim}" />
-  </joint>
+      </visual>
+      <collision>
+        <origin xyz="0 0 0" rpy="${pi/2} 0 0"/>
+          <geometry>
+            <cylinder radius="${wheel_radius}" length="${wheel_thickness}"/>
+          </geometry>
+      </collision>
+      <xacro:disk_inertia mass="${wheel_mass}" radius="${wheel_radius}" height="${wheel_thickness}">
+        <origin xyz="0 0 0" rpy="${-pi/2} 0 0" />
+      </xacro:disk_inertia >
+    </link>
+  </xacro:macro>
 </robot>

Commit message: progresses on testing horizon

File: wheebbot_description/urdf/gazebo_spec_tags.xacro (robot description, xacro)
@@ -105,19 +105,16 @@
   </gazebo>
   <!-- diff drive plugin -->
-  <!-- <gazebo>
+<!--
+  <gazebo>
     <plugin name='diff_drive' filename='libgazebo_ros_diff_drive.so'>
       <ros>
         <namespace>/base_state</namespace>
       </ros>
-      <!-- wheels -->
       <left_joint>left_wheel_joint</left_joint>
       <right_joint>right_wheel_joint</right_joint>
-      <!-- kinematics -->
       <wheel_separation> 0.028</wheel_separation>
       <wheel_diameter> 0.12 </wheel_diameter>
-      <!-- limits -->
       <max_wheel_torque>2</max_wheel_torque>
       <max_wheel_acceleration>1.0</max_wheel_acceleration>
-      <!-- output -->
       <publish_odom>true</publish_odom>
       <publish_odom_tf>false</publish_odom_tf>

File: wheebbot_description/urdf/wheebbot.urdf (robot description, URDF)
Before this commit: robot wheebbot_full, 4 links, 3 joints
Links:
- removed link aux_link
- removed link body
- removed link left_wheel
- removed link right_wheel
Joints:
- removed joint aux_joint
- removed joint left_wheel_joint
- removed joint right_wheel_joint

File: wheebbot_description/urdf/wheebbot_full.urdf.xacro (robot description, xacro)
@@ -7,5 +7,5 @@
         <link name="world">
         </link>
-        <joint name="world2wheebbot" type="floating">
+        <joint name="world_jnt" type="floating">
             <origin xyz="0 0 0" rpy="0 0 0"/>
             <parent link="world"/>
@@ -13,6 +13,4 @@
         </joint>
     </xacro:if>
-    <xacro:unless value="$(arg is_floating_base)">
-    </xacro:unless>
     <!-- Generating wheebbot description based on the arguments -->
     <xacro:ign_or_gazebo is_gazebo_classic="$(arg is_gazebo_classic)"/>
