Commit message: small update

File: wheebbot_description/urdf/gazebo_spec_tags.xacro (robot description, xacro)
@@ -2,5 +2,5 @@
 <robot xmlns:xacro="http://www.ros.org/wiki/xacro">
   <xacro:property name="yaml_file" value="$(find wheebbot_description)/config/urdf_params.yaml" />
-  <xacro:property name="props" value="${load_yaml(yaml_file)}"/>
+  <xacro:property name="props" value="${xacro.load_yaml(yaml_file)}"/>
   <xacro:property name="wheels_interax" value="${props['wheebbot']['wheels_interax']}" />
   <xacro:property name="wheels_diameter" value="${2* props['wheebbot']['wheel_radius']}" />

File: wheebbot_description/urdf/generated/wheebbot_full.urdf (robot description, URDF)
Before this commit: robot wheebbot_full, 5 links, 4 joints
Links:
- removed link world
Joints:
- removed joint world_jnt
- joint left_wheel_joint: limit lower=-inf upper=inf effort=30.0 velocity=100.0 -> lower=-1e+25 upper=1e+25 effort=30.0 velocity=100.0
- joint right_wheel_joint: limit lower=-inf upper=inf effort=30.0 velocity=100.0 -> lower=-1e+25 upper=1e+25 effort=30.0 velocity=100.0

File: wheebbot_description/urdf/parameters.urdf.xacro (robot description, xacro)
@@ -3,5 +3,5 @@
   <!-- Reading some parameters from a YAML config file -->
   <xacro:property name="yaml_file" value="$(find wheebbot_description)/config/urdf_params.yaml" />
-  <xacro:property name="props" value="${load_yaml(yaml_file)}"/>
+  <xacro:property name="props" value="${xacro.load_yaml(yaml_file)}"/>
   <!-- Assigning those parameters to xacro properties -->
   <xacro:property name="pendulum_mass" value="${props['wheebbot']['pendulum_mass']}" />

File: wheebbot_description/urdf/wheebbot.urdf.xacro (robot description, xacro)
@@ -1,5 +1,5 @@
 <?xml version="1.0"?>
 <robot name="wheebbot" xmlns:xacro="http://www.ros.org/wiki/xacro">
-  <xacro:macro name="ign_or_gazebo" params="is_gazebo_classic" >
+  <xacro:macro name="ign_or_gazebo" params="is_gazebo_classic:=false" >
     <!-- Including the parameters file -->
     <xacro:include filename="$(find wheebbot_description)/urdf/parameters.urdf.xacro" />
@@ -29,5 +29,5 @@
         <origin xyz="0 ${box_ly/2-leg_extrusion_l_edge/2} ${-(box_lz/2-leg_extrusion_l_edge/2)}" rpy="0 0 ${-pi/2}" />
         <geometry>
-          <mesh filename="package://wheebbot_description/meshes/full_no_knee_no_wheels.dae" scale="1.0 1.0 1.0" />
+          <mesh filename="package://wheebbot_description/urdf/meshes/full_no_knee_no_wheels.dae" scale="1.0 1.0 1.0" />
         </geometry>
       </visual>
@@ -125,5 +125,5 @@
         <origin xyz="0 0 0" rpy="0 0 ${pi/2}" />
         <geometry>
-          <mesh filename="package://wheebbot_description/meshes/wheel_black.dae" scale="1.0 1.0 1.0" />
+          <mesh filename="package://wheebbot_description/urdf/meshes/wheel_black.dae" scale="1.0 1.0 1.0" />
         </geometry>
       </visual>
@@ -151,5 +151,5 @@
         <origin xyz="0 0 0" rpy="0 0 ${-pi/2}" />
         <geometry>
-          <mesh filename="package://wheebbot_description/meshes/wheel_black.dae" scale="1.0 1.0 1.0" />
+          <mesh filename="package://wheebbot_description/urdf/meshes/wheel_black.dae" scale="1.0 1.0 1.0" />
         </geometry>
       </visual>

File: wheebbot_description/urdf/wheebbot_full.urdf.xacro (robot description, xacro)
@@ -1,6 +1,6 @@
 <?xml version="1.0"?>
 <robot name="wheebbot_full" xmlns:xacro="http://www.ros.org/wiki/xacro">
-    <xacro:arg name="is_gazebo_classic" default="true" />
-    <xacro:arg name="is_floating_base" default="true" />
+    <xacro:arg name="is_gazebo_classic" default="false" />
+    <xacro:arg name="is_floating_base" default="false" />
     <xacro:include filename="$(find wheebbot_description)/urdf/wheebbot.urdf.xacro" />
     <xacro:if value="$(arg is_floating_base)">
