Commit message: moved from continuous joint to revolute to avoid pinocchio cos, sin representation

File: wheebbot_description/urdf/generated/wheebbot_full.urdf (robot description, URDF)
Before this commit: robot wheebbot_full, 4 links, 3 joints
Links:
- added link world
Joints:
- added joint world_jnt: type floating, parent world, child aux_link, origin xyz=0 0 0 rpy=0 0 0
- joint left_wheel_joint: limit effort=30.0 velocity=100.0 -> lower=-inf upper=inf effort=30.0 velocity=100.0; type continuous -> revolute
- joint right_wheel_joint: limit effort=30.0 velocity=100.0 -> lower=-inf upper=inf effort=30.0 velocity=100.0; type continuous -> revolute

File: wheebbot_description/urdf/parameters.urdf.xacro (robot description, xacro)
@@ -43,3 +43,4 @@
   <xacro:property name="door_handle_lenght2" value="${props['wheebbot']['door_handle_lenght2']}" />
   <xacro:property name="door_handle_width" value="${props['wheebbot']['door_handle_width']}" />
+   <xacro:property name="big_joint_limit" value="${1e25}" />
 </robot>

File: wheebbot_description/urdf/wheebbot.urdf.xacro (robot description, xacro)
@@ -112,5 +112,5 @@
       </xacro:box_inertia>
     </link>
-    <joint name="left_wheel_joint" type="continuous">
+    <joint name="left_wheel_joint" type="revolute">
       <origin xyz="0 ${(wheels_interax/2)} ${-(box_lz/2+leg_length+motor_case_l_edge/2)}" rpy="0 0 0"/>
       <parent link="body"/>
@@ -118,5 +118,5 @@
       <axis xyz="0 1 0" />
       <dynamics damping="${wheel_joint_damping}" friction="${wheel_joint_static_friction}"/>
-      <limit effort="${wheel_joint_effort_lim}" velocity="${wheel_joint_velocity_lim}" />
+      <limit effort="${wheel_joint_effort_lim}" velocity="${wheel_joint_velocity_lim}" lower="-${big_joint_limit}" upper="${big_joint_limit}" />
     </joint>
     <link name="left_wheel">
@@ -138,5 +138,5 @@
       </xacro:disk_inertia>
     </link>
-    <joint name="right_wheel_joint" type="continuous">
+    <joint name="right_wheel_joint" type="revolute">
       <origin xyz="0 ${-(wheels_interax/2)} ${-(box_lz/2+leg_length+motor_case_l_edge/2)}" rpy="0 0 0"/>
       <parent link="body"/>
@@ -144,5 +144,5 @@
       <axis xyz="0 1 0" />
       <dynamics damping="${wheel_joint_damping}" friction="${wheel_joint_static_friction}"/>
-      <limit effort="${wheel_joint_effort_lim}" velocity="${wheel_joint_velocity_lim}" />
+      <limit effort="${wheel_joint_effort_lim}" velocity="${wheel_joint_velocity_lim}" lower="-${big_joint_limit}" upper="${big_joint_limit}" />
     </joint>
     <link name="right_wheel">

File: wheebbot_description/urdf/wheebbot_full.urdf.xacro (robot description, xacro)
@@ -2,5 +2,5 @@
 <robot name="wheebbot_full" xmlns:xacro="http://www.ros.org/wiki/xacro">
     <xacro:arg name="is_gazebo_classic" default="true" />
-    <xacro:arg name="is_floating_base" default="false" />
+    <xacro:arg name="is_floating_base" default="true" />
     <xacro:include filename="$(find wheebbot_description)/urdf/wheebbot.urdf.xacro" />
     <xacro:if value="$(arg is_floating_base)">
